File: hardware/flex-fule-can-adapter-v1/flex-fule-can-adapter-v1.kicad_pcb (KiCad board)
At the start: 2 copper layers, 60 x 35 mm, 52 parts, among them J1 1565749-4, J2 1565749-4, J3 USB4520-03-1-A, SW1 RESET, SW2 BOOT, U1 ESP32-C3-WROOM-02U-N4, U2 SN65HVD230QDR, U3 TPS259472ARPWR, U4 TPS62901RPJR, U5 USBLC6-2SC6

Commit message: Late night final push. review in morning*
Parts:
- removed C19: 10nF, Capacitor_SMD:C_0603_1608Metric
- removed C21: 10uF 25V, Capacitor_SMD:C_0603_1608Metric
- removed C22: 22uF, Capacitor_SMD:C_0603_1608Metric
- removed J3: USB4520-03-1-A, flex-fule:USB4520031A
- removed JP1: PWR_SEL, Jumper:SolderJumper-3_P1.3mm_Open_RoundedPad1.0x1.5mm_NumberLabels
- removed L3: F1C1-201612-2R2M, flex-fule:F1C12016122R2M
- removed R13: 5.1k, Resistor_SMD:R_0603_1608Metric
- removed R16: 113k, Resistor_SMD:R_0603_1608Metric
- removed R17: 24.9k, Resistor_SMD:R_0603_1608Metric
- removed U5: USBLC6-2SC6, Package_TO_SOT_SMD:SOT-23-6
- added C10: 22uF, Capacitor_SMD:C_0603_1608Metric_Pad1.08x0.95mm_HandSolder, F.Cu at (127.4, 118.8)
- added C11: 22uF, Capacitor_SMD:C_0603_1608Metric_Pad1.08x0.95mm_HandSolder, F.Cu at (127.4, 122.5)
- added C8: 100nF, Capacitor_SMD:C_0603_1608Metric_Pad1.08x0.95mm_HandSolder, F.Cu at (135.3, 124.0)
- added C9: 10uF, Capacitor_SMD:C_0603_1608Metric_Pad1.08x0.95mm_HandSolder, F.Cu at (132.1, 127.3)
- added D+: D+, TestPoint:TestPoint_Pad_D2.0mm, F.Cu at (122.0, 131.0)
- added D-: D-, TestPoint:TestPoint_Pad_D2.0mm, F.Cu at (126.0, 131.0)
- added L1: PA4332.332NLT, flex-fule:PA4332332NLT, F.Cu at (132.1, 119.8)
- R12: value 5.1k -> 0; footprint Resistor_SMD:R_0603_1608Metric -> Resistor_SMD:R_0603_1608Metric_Pad0.98x0.95mm_HandSolder
- U4: value TPS62901RPJR -> AP63203QWU-7; footprint flex-fule:TPS62901RPJR -> flex-fule:SOT95P280X100-6N
- moved R12 78.5 mm to (117.6, 122.7), turned to -90 degrees
- moved R3 64.6 mm to (126.3, 127.0), turned to 90 degrees
- moved R4 61.5 mm to (128.1, 127.0), turned to 90 degrees
- moved C3 54.5 mm to (136.4, 127.0), turned to 180 degrees
- moved C1 51.0 mm to (137.8, 118.8), turned to -90 degrees
- moved C2 49.8 mm to (135.9, 118.8), turned to -90 degrees
- moved R2 41.9 mm to (140.6, 106.8)
- moved R1 40.9 mm to (137.4, 124.0), turned to 90 degrees
- moved R14 34.2 mm to (148.0, 104.4), turned to 180 degrees
- moved R15 33.9 mm to (148.0, 106.4), turned to 180 degrees
- moved R19 33.6 mm to (148.0, 108.5), turned to 180 degrees
- moved LED1 31.6 mm to (154.0, 108.3), turned to -90 degrees
- moved SW1 17.3 mm to (134.1, 130.2), turned to 0 degrees
- moved R18 17.1 mm to (148.3, 126.8), turned to 0 degrees
- moved LED2 16.8 mm to (153.1, 126.8), turned to 180 degrees
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Connections:
- net /PWR_LED renamed Net-(LED2-A)
- R12 pad 1: GND -> VBAT
- R12 pad 2: Net-(J3-CC1) -> 12V
- R14 pad 2: unconnected-(R14-Pad2) -> Net-(U1-IO7)
- R15 pad 2: Net-(U1-IO5) -> Net-(U1-IO6)
- R19 pad 2: Net-(U1-IO6) -> Net-(U1-IO5)
- U1 pad 6: unconnected-(U1-IO7-Pad6) -> Net-(U1-IO7)
- U4 pad 1: unconnected-(U4-PG-Pad1) -> 3.3V
- U4 pad 2: Net-(U4-SW) -> 12V
- U4 pad 3: 3.3V -> 12V
- U4 pad 5: Net-(JP1-C) -> Net-(U4-SW)
- U4 pad 6: Net-(JP1-C) -> Net-(U4-BST)
Routing:
- net 3.3V: track 12.8 -> 115.0 mm, vias 0 -> 5
- net Net-(U1-IO9): track 0.00 -> 27.7 mm
- net 12V: track 6.33 -> 30.9 mm, vias 0 -> 3
- net Net-(U1-IO18): track 0.00 -> 22.5 mm, vias 0 -> 2
- net Net-(U1-IO19): track 0.00 -> 20.3 mm, vias 0 -> 2
- net Net-(U1-EN): track 0.00 -> 20.2 mm
- net Net-(U1-IO7): track 0.00 -> 14.7 mm, vias 0 -> 2
- net Net-(U1-IO6): track 0.00 -> 14.5 mm, vias 0 -> 2
- net Net-(U1-IO5): track 0.00 -> 14.3 mm, vias 0 -> 2
- net GND: track 11.2 -> 24.8 mm, vias 2 -> 51
- net VBUS: track 13.0 -> 0.00 mm
- net VBAT: track 12.4 -> 22.8 mm
- net Net-(JP1-C): track 8.10 -> 0.00 mm
- net Net-(LED1-B): track 0.00 -> 6.83 mm
- net Net-(LED1-R): track 0.00 -> 6.35 mm
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- added copper zone on B.Cu, net GND
- added copper zone on F.Cu, net GND
Other:
- board size 60 x 35 mm -> 55 x 31 mm

Commit message: ready for production
Parts:
- added REF**: Untitled, Untitled, F.Cu at (142.1, 124.7)
- added REF**: Untitled, Untitled, F.Cu at (107.3, 127.3)
- added TP1: TestPoint, TestPoint:TestPoint_Pad_D1.0mm, F.Cu at (117.4, 116.3)
- added TP2: TestPoint, TestPoint:TestPoint_Pad_D1.0mm, F.Cu at (117.4, 114.0)
- added TP3: TestPoint, TestPoint:TestPoint_Pad_D1.0mm, F.Cu at (117.4, 111.7)
Connections:
- U1 pad 15: unconnected-(U1-IO3-Pad15) -> Net-(U1-IO3)
- U1 pad 17: unconnected-(U1-IO1-Pad17) -> Net-(U1-IO1)
- U1 pad 18: unconnected-(U1-IO0-Pad18) -> Net-(U1-IO0)
Routing:
- net Net-(U1-IO0): track 0.00 -> 2.76 mm
- net Net-(U1-IO3): track 0.00 -> 2.72 mm
- net Net-(U1-IO1): track 0.00 -> 2.43 mm
- net /CAN-: track 15.1 -> 16.0 mm
- net GND: vias 51 -> 76
Other:
- board text added: "FFCA V1.0"
- board text added: "Flex Fule Adapter"
