File: hardware/flex-fule-can-adapter-v1/flex-fule-can-adapter-v1.kicad_sch (KiCad schematic)
At the start: 38 parts, among them J1 Ethanol Sensor, J2 CAR, SW1 RESET, SW2 BOOT, U1 ESP32-C3-WROOM-02U-N4, U2 SN65HVD230QDR, U3 TPS259472ARPWR, U4 TPS62901RPJR

Commit message: Sch done
Parts:
- added D3: ESDCAN03-2BWY, SDM_MiscFootprint:SOT65P210X110-3N, symbol SDM_DIODES:ESDCAN03-2BWY
- added J3: USB4520-03-1-A, ModLib:USB4520031A, symbol SchLib:USB4520-03-1-A
- added JP1: PWR_SEL, Jumper:SolderJumper-3_P1.3mm_Open_RoundedPad1.0x1.5mm_NumberLabels, symbol Jumper:SolderJumper_3_Open
- added R12, R13: 5.1k, Resistor_SMD:R_0603_1608Metric, symbol Device:R
- added U5: USBLC6-2SC6, Package_TO_SOT_SMD:SOT-23-6, symbol Power_Protection:USBLC6-2SC6
Connections:
- net 12V: now also JP1.1 (A); no longer C21.1, C7.1, U3.6 (OUT), U4.5 (EN), U4.6 (VIN)
- net CAN+: now also D3.2
- net CAN-: now also D3.1
- net GND: now also D3.3, J3.A1 (GND_1), J3.A12 (GND_2), J3.MH1, J3.MH2, J3.MH3, J3.MH4, R12.1, R13.1, U5.2 (GND)
- net USB_D+: now also U5.1 (I/O1)
- net USB_D-: now also U5.3 (I/O2)
- net Eth_inp: now reaches R7.2
- net Eth_inp: now also U1.4 (IO5)
- new net: J3.A7 (DN1), J3.B7 (DN2), U5.4 (I/O2)
- new net: J3.A6 (DP1), J3.B6 (DP2), U5.6 (I/O1)
- new net: C21.1, C7.1, JP1.2 (C), U3.6 (OUT), U4.5 (EN), U4.6 (VIN)
- new net: J3.A5 (CC1), R12.2
- new net: J3.B5 (CC2), R13.2
- new net VBUS: J3.A4 (VBUS_1), J3.A9 (VBUS_2), JP1.3 (B), U5.5 (VBUS)
- no-connect marks 8 -> 10
Other:
- note added: "CONN"
- moved on the sheet: C1, C19, C2, C21, C22, C23, C24, C3, C4, C5, C6, C7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

Commit message: PCB progress
Parts:
- removed J1: Ethanol Sensor, symbol Connector:Conn_01x03_Pin
- removed J2: CAR, symbol Connector:Conn_01x04_Pin
- added H1, H2, H3, H4: MH, MountingHole:MountingHole_2.2mm_M2_Pad_Via, symbol Mechanical:MountingHole_Pad
- added J1, J2: 1565749-4, flex-fule:15657494, symbol flex-fule:1565749-4
- added LED1: CLMUD-FKC-CHJNPM569ABB845343, flex-fule:PLCC4_CLMUD-FKC_CRW-L, symbol LED:APFA3010
- added R14: 330, Resistor_SMD:R_0603_1608Metric_Pad0.98x0.95mm_HandSolder, symbol Device:R_Small
- added R15, R19: 150, Resistor_SMD:R_0603_1608Metric_Pad0.98x0.95mm_HandSolder, symbol Device:R_Small
- C6, C7: footprint (none) -> Capacitor_SMD:C_0603_1608Metric_Pad1.08x0.95mm_HandSolder
- D1: footprint TPD1E10B06DPYT:DIO_TPD1E05U06DPYR -> flex-fule:DIO_TPD1E05U06DPYR
- D2: footprint DIOM5436X244N -> flex-fule:DIOM5436X244N
- D3: footprint SDM_MiscFootprint:SOT65P210X110-3N -> flex-fule:SOT65P210X110-3N
- J3: footprint ModLib:USB4520031A -> flex-fule:USB4520031A
- L3: footprint F1C12016122R2M -> flex-fule:F1C12016122R2M
- SW1, SW2: footprint (none) -> Button_Switch_SMD:SW_SPST_CK_RS282G05A3
- U1: footprint ESP32-C3-WROOM-02U-N4:XCVR_ESP32-C3-WROOM-02U-N4 -> flex-fule:XCVR_ESP32-C3-WROOM-02U-N4
- U2: footprint SOIC127P600X175-8N -> flex-fule:SOIC127P600X175-8N
- U3: footprint TPS259472ARPWR -> flex-fule:TPS259472ARPWR
- U4: footprint TPS62901RPJR -> flex-fule:TPS62901RPJR
Connections:
- net 12V: now also C7.1, U3.6 (OUT), J1.4
- net 3.3V: now also LED1.1 (A)
- net CAN+: now also J2.3
- net CAN-: now also J2.4
- net CAN_RX: now also U1.11 (IO20); no longer U1.17 (IO1)
- net CAN_TX: now also U1.12 (IO21); no longer U1.18 (IO0)
- net Eth_inp: now also U1.3 (IO4); no longer U1.4 (IO5)
- net GND: now also H1.1, H2.1, H3.1, H4.1, J1.1, J1.3, J1.MH1, J1.MH2, J2.2, J2.MH1, J2.MH2
- net VBAT: now also J2.1
- net at C21.1, JP1.2 (C), U4.5 (EN)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: no longer C7.1, U3.6 (OUT)
- net at D1.2, R6.1, R7.1: now also J1.2
- net at U1.5 (IO6): now also R19.2
- new net: LED1.2 (R), R14.1
- new net: R15.2, U1.4 (IO5)
- new net: LED1.4 (B), R19.1
- new net: LED1.3 (G), R15.1
Other:
- moved on the sheet: C1, C19, C2, C21, C22, C23, C24, C3, C4, C5, C6, C7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

Commit message: Late night final push. review in morning*
Parts:
- removed C19: 10nF, Capacitor_SMD:C_0603_1608Metric, symbol Device:C_Small
- removed C21: 10uF 25V, Capacitor_SMD:C_0603_1608Metric, symbol Device:C_Small
- removed C22: 22uF, Capacitor_SMD:C_0603_1608Metric, symbol Device:C_Small
- removed J3: USB4520-03-1-A, flex-fule:USB4520031A, symbol SchLib:USB4520-03-1-A
- removed JP1: PWR_SEL, Jumper:SolderJumper-3_P1.3mm_Open_RoundedPad1.0x1.5mm_NumberLabels, symbol Jumper:SolderJumper_3_Open
- removed L3: F1C1-201612-2R2M, flex-fule:F1C12016122R2M, symbol SDM_MISC:F1C1-201612-2R2M
- removed R12, R13: 5.1k, Resistor_SMD:R_0603_1608Metric, symbol Device:R
- removed R16: 113k, Resistor_SMD:R_0603_1608Metric, symbol Device:R_Small
- removed R17: 24.9k, Resistor_SMD:R_0603_1608Metric, symbol Device:R_Small
- removed U4: TPS62901RPJR, flex-fule:TPS62901RPJR, symbol SDM_MISC:TPS62901RPJR
- removed U5: USBLC6-2SC6, Package_TO_SOT_SMD:SOT-23-6, symbol Power_Protection:USBLC6-2SC6
- added C10, C11: 22uF, Capacitor_SMD:C_0603_1608Metric_Pad1.08x0.95mm_HandSolder, symbol Device:C_Small
- added C8: 100nF, Capacitor_SMD:C_0603_1608Metric_Pad1.08x0.95mm_HandSolder, symbol Device:C_Small
- added C9: 10uF, Capacitor_SMD:C_0603_1608Metric_Pad1.08x0.95mm_HandSolder, symbol Device:C_Small
- added D+1: D+, TestPoint:TestPoint_Pad_D2.0mm, symbol Connector:TestPoint
- added D-1: D-, TestPoint:TestPoint_Pad_D2.0mm, symbol Connector:TestPoint
- added L1: PA4332.332NLT, PA4332332NLT, symbol flex-fule:PA4332.332NLT
- added R12: 0, Resistor_SMD:R_0603_1608Metric_Pad0.98x0.95mm_HandSolder, symbol Device:R_Small
- added U4: AP63203QWU-7, SOT95P280X100-6N, symbol flex-fule:AP63203QWU-7
Connections:
- net 12V: now also C9.1, R12.2, U4.2 (EN), U4.3 (VIN)
- net 3.3V: now also C10.1, C11.1, L1.2, U4.1 (FB)
- net GND: now also C10.2, C11.2, C9.2, U4.4 (GND)
- net USB_D+: now also D+1.1
- net USB_D-: now also D-1.1
- net VBAT: now also R12.1
- net at R14.2: now also U1.6 (IO7)
- net at U1.4 (IO5): now also R19.2; no longer R15.2
- net at U1.5 (IO6): now also R15.2; no longer R19.2
- net PWR_LED: no longer names the net of LED2.2 (A), R18.2
- new net: C8.2, L1.1, U4.5 (SW)
- new net: C8.1, U4.6 (BST)
- no-connect marks 10 -> 6
Other:
- moved on the sheet: C23, C24, C6, C7, D2, R10, R11, R8, R9, U3

Commit message: ready for production
Parts:
- added TP1, TP2, TP3: TestPoint, TestPoint:TestPoint_Pad_D1.5mm, symbol Connector:TestPoint
Connections:
- net at U1.15 (IO3): now also TP3.1
- net at U1.17 (IO1): now also TP2.1
- net at U1.18 (IO0): now also TP1.1
Changed lines of the file:
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@@
 	)
 	(symbol
+		(lib_id "Connector:TestPoint")
+		(at 132.08 48.26 270)
+		(unit 1)
+		(body_style 1)
+		(exclude_from_sim no)
+		(in_bom yes)
+		(on_board yes)
+		(in_pos_files yes)
+		(dnp no)
+		(property "Reference" "TP1"
+			(at 132.334 47.498 90)
+			(show_name no)
+			(do_not_autoplace no)
+			(effects
+				(font
+					(size 0.762 0.762)
+				)
+				(justify left)
+			)
+		)
+		(property "Value" "TestPoint"
+			(at 136.398 48.006 90)
+			(show_name no)
+			(do_not_autoplace no)
+			(effects
+				(font
+					(size 0.762 0.762)
+				)
+				(justify left)
+			)
+		)
+		(property "Footprint" "TestPoint:TestPoint_Pad_D1.5mm"
+			(at 132.08 53.34 0)
+			(hide yes)
+			(show_name no)
+			(do_not_autoplace no)
+			(effects
+				(font
+					(size 1.27 1.27)
+				)
+			)
+		)
+		(property "Datasheet" ""
+			(at 132.08 53.34 0)
+			(hide yes)
+			(show_name no)
+			(do_not_autoplace no)
+			(effects
+				(font
+					(size 1.27 1.27)
+				)
+			)
+		)
+		(property "Description" "test point"
+			(at 132.08 48.26 0)
+			(hide yes)
+			(show_name no)
+			(do_not_autoplace no)
+			(effects
+				(font
+					(size 1.27 1.27)
+				)
+			)
+		)
+		(pin "1"
+		)
+		(instances
+			(project "flex-fule-can-adapter-v1"
+				(path "/077978c9-a704-4aa8-820f-9f7a9583649a"
+					(reference "TP1")
+					(unit 1)
+				)
+			)
+		)
+	)
+	(symbol
 		(lib_id "power:GND")
 		(at 204.47 109.22 0)
@@
 	)
 	(symbol
+		(lib_id "Connector:TestPoint")
+		(at 132.08 53.34 270)
+		(unit 1)
+		(body_style 1)
+		(exclude_from_sim no)
+		(in_bom yes)
+		(on_board yes)
+		(in_pos_files yes)
+		(dnp no)
+		(property "Reference" "TP3"
+			(at 132.334 52.578 90)
+			(show_name no)
+			(do_not_autoplace no)
+			(effects
+				(font
+					(size 0.762 0.762)
+				)
+				(justify left)
+			)
+		)
+		(property "Value" "TestPoint"
+			(at 136.398 53.086 90)
+			(show_name no)
+			(do_not_autoplace no)
+			(effects
+				(font
+					(size 0.762 0.762)
+				)
+				(justify left)
+			)
+		)
+		(property "Footprint" "TestPoint:TestPoint_Pad_D1.5mm"
+			(at 132.08 58.42 0)
+			(hide yes)
+			(show_name no)
+			(do_not_autoplace no)
+			(effects
+				(font
+					(size 1.27 1.27)
+				)
+			)
+		)
+		(property "Datasheet" ""
+			(at 132.08 58.42 0)
+			(hide yes)
+			(show_name no)
+			(do_not_autoplace no)
+			(effects
+				(font
+					(size 1.27 1.27)
+				)
+			)
+		)
+		(property "Description" "test point"
+			(at 132.08 53.34 0)
+			(hide yes)
+			(show_name no)
+			(do_not_autoplace no)
+			(effects
+				(font
+					(size 1.27 1.27)
+				)
+			)
+		)
+		(pin "1"
+		)
+		(instances
+			(project "flex-fule-can-adapter-v1"
+				(path "/077978c9-a704-4aa8-820f-9f7a9583649a"
+					(reference "TP3")
+					(unit 1)
+				)
+			)
+		)
+	)
+	(symbol
 		(lib_id "Device:C_Small")
 		(at 62.23 129.54 0)
@@
 					(unit 1)
 				)
+			)
+		)
+	)
+	(symbol
+		(lib_id "Connector:TestPoint")
+		(at 132.08 50.8 270)
+		(unit 1)
+		(body_style 1)
+		(exclude_from_sim no)
+		(in_bom yes)
+		(on_board yes)
+		(in_pos_files yes)
+		(dnp no)
+		(property "Reference" "TP2"
+			(at 132.334 50.038 90)
+			(show_name no)
+			(do_not_autoplace no)
+			(effects
+				(font
+					(size 0.762 0.762)
+				)
+				(justify left)
+			)
+		)
+		(property "Value" "TestPoint"
+			(at 136.398 50.546 90)
+			(show_name no)
+			(do_not_autoplace no)
+			(effects
+				(font
+					(size 0.762 0.762)
+				)
+				(justify left)
+			)
+		)
+		(property "Footprint" "TestPoint:TestPoint_Pad_D1.5mm"
+			(at 132.08 55.88 0)
+			(hide yes)
+			(show_name no)
+			(do_not_autoplace no)
+			(effects
+				(font
+					(size 1.27 1.27)
+				)
+			)
+		)
+		(property "Datasheet" ""
+			(at 132.08 55.88 0)
+			(hide yes)
+			(show_name no)
+			(do_not_autoplace no)
+			(effects
+				(font
+					(size 1.27 1.27)
+				)
+			)
+		)
+		(property "Description" "test point"
+			(at 132.08 50.8 0)
+			(hide yes)
+			(show_name no)
+			(do_not_autoplace no)
+			(effects
+				(font
+					(size 1.27 1.27)
+				)
+			)
+		)
+		(pin "1"
+		)
+		(instances
+			(project "flex-fule-can-adapter-v1"
+				(path "/077978c9-a704-4aa8-820f-9f7a9583649a"
+					(reference "TP2")
+					(unit 1)
+				)
